File: PCB/New folder/foc_terminal_ver/foc_terminal_ver.kicad_pcb (KiCad board)
At the start: 4 copper layers, 50 x 50 mm, 100 parts, among them J1 SWD, J2 USB_C_Receptacle_USB2.0_16P, J3 Conn_02x09_Odd_Even, J4 XT30PW_2_2_-M.G.B, J8 XT30PW_2_2_-M.G.B, J9 Conn_01x05, Q1 DON50N04, Q2 DON50N04, Q3 DON50N04, Q4 NMOS-8PINS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

Commit message: update
Parts:
- removed J4: XT30PW_2_2_-M.G.B, XT30PW_2_2_-M.G.B:AMASS_XT30PW_2_2_-M.G.B
- added J6: CAN_OUT, Connector_JST:JST_GH_SM04B-GHS-TB_1x04-1MP_P1.25mm_Horizontal, F.Cu at (123.0, 108.5)
- added J7: CAN_IN, Connector_JST:JST_GH_SM04B-GHS-TB_1x04-1MP_P1.25mm_Horizontal, F.Cu at (123.0, 118.0)
- moved D2 86.1 mm to (107.1, 111.7)
- moved D4 86.1 mm to (107.1, 113.2)
- moved D5 86.1 mm to (107.1, 114.7)
- moved R11 86.1 mm to (110.1, 113.2)
- moved R12 86.1 mm to (110.1, 114.7)
- moved R8 86.1 mm to (110.1, 111.7)
- moved J8 83.9 mm to (199.2, 95.2), turned to 90 degrees
- moved J1 70.9 mm to (121.9, 102.0)
- moved JP3 23.0 mm to (116.7, 120.9)
- moved JP5 23.0 mm to (116.7, 123.5)
Routing:
- net SWDIO: track 0.00 -> 18.7 mm
- net SWCLK: track 0.00 -> 18.1 mm
- net CAN_H: track 0.00 -> 11.5 mm
