File: PCB/New folder/foc_terminal_ver/foc_terminal_ver.kicad_sch (KiCad schematic)
At the start: 103 parts, among them J1 SWD, J2 USB_C_Receptacle_USB2.0_16P, J3 Conn_02x09_Odd_Even, J4 XT30PW_2_2_-M.G.B, J6 CAN_OUT, J7 CAN_IN, J8 XT30PW_2_2_-M.G.B, J9 Conn_01x05, Q1 DON50N04, Q2 DON50N04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

Commit message: update
Parts:
- removed J4: XT30PW_2_2_-M.G.B, XT30PW_2_2_-M.G.B:AMASS_XT30PW_2_2_-M.G.B, symbol XT30PW_2_2_-M.G.B:XT30PW_2_2_-M.G.B
Other:
- moved on the sheet: J6, J7
