File: PCB/foc-motor-controller.kicad_pcb (KiCad board)
At the start: 4 copper layers, 50 x 50 mm, 100 parts, among them J1 SWD, J2 USB_C_Receptacle_USB2.0_16P, J3 Conn_02x09_Odd_Even, J4 XT30PW_2_2_-M.G.B, J8 XT30PW_2_2_-M.G.B, J9 Conn_01x05, Q1 DON50N04, Q2 DON50N04, Q3 DON50N04, Q4 NMOS-8PINS, Q5 DON50N04, Q6 DON50N04, U1 MT6826SGT, U2 STM32G431RBTx, U3 DRV8323SRTAT, U4 MIC5219-3.3YM5, U5 TCAN1044V, U6 USBLC6-2SC6, U7 TPS54240DGQ, Y1 Resonator

Commit message: update
Parts:
- removed C35: 22uF, Capacitor_SMD:C_0805_2012Metric
- removed J9: Conn_01x05, TiManh:TerminalBlock_1x05_P6.35mm_Horizontal
- removed U6: USBLC6-2SC6, Package_TO_SOT_SMD:SOT-23-6
- added C12: 100nF, Capacitor_SMD:C_0603_1608Metric, F.Cu at (151.2, 121.8)
- added C20: 100nF, Capacitor_SMD:C_0603_1608Metric, F.Cu at (155.8, 121.8)
- added C40: C_Polarized, Capacitor_SMD:CP_Elec_6.3x5.9, F.Cu at (135.0, 94.0)
- added C41: 10uF, Capacitor_SMD:C_1206_3216Metric, F.Cu at (156.0, 94.0)
- added C42: 10uF, Capacitor_SMD:C_1206_3216Metric, F.Cu at (158.3, 94.0)
- added C43: 10uF, Capacitor_SMD:C_1206_3216Metric, F.Cu at (139.7, 94.0)
- added C44: 10uF, Capacitor_SMD:C_1206_3216Metric, F.Cu at (142.0, 94.0)
- added C45: 10uF, Capacitor_SMD:C_1206_3216Metric, F.Cu at (144.3, 94.0)
- added D3: D_TVS, Diode_SMD:D_SMB, F.Cu at (128.5, 93.8)
- added J6: Conn_01x08, Connector_JST:JST_GH_SM08B-GHS-TB_1x08-1MP_P1.25mm_Horizontal, F.Cu at (155.0, 127.0)
- added JP1: Jumper_3_Open, Jumper:SolderJumper-3_P1.3mm_Open_RoundedPad1.0x1.5mm, B.Cu at (147.2, 123.8)
- added R10: 10K, Resistor_SMD:R_0603_1608Metric, F.Cu at (154.7, 100.6)
- added R27: 47R, Resistor_SMD:R_0603_1608Metric, F.Cu at (152.7, 121.8)
- added R28: 4.7K, Resistor_SMD:R_0603_1608Metric, F.Cu at (158.8, 121.8)
- added R29: 4.7K, Resistor_SMD:R_0603_1608Metric, F.Cu at (157.3, 121.8)
- added TH1: Thermistor_NTC, Resistor_SMD:R_0603_1608Metric, B.Cu at (153.2, 96.2)
- added TP6: TestPoint, TestPoint:TestPoint_Pad_D1.0mm, B.Cu at (145.0, 109.1)
- added TP7: TestPoint, TestPoint:TestPoint_Pad_D1.0mm, B.Cu at (143.0, 109.1)
- added TP8: TestPoint, TestPoint:TestPoint_Pad_D1.0mm, B.Cu at (147.0, 109.1)
- C22, C25: value 470uF -> C_Polarized; footprint Capacitor_SMD:C_Elec_10x10.2 -> Capacitor_SMD:CP_Elec_6.3x5.9
- C34: value 470uF -> 10uF; footprint Capacitor_SMD:C_Elec_10x10.2 -> Capacitor_SMD:C_1206_3216Metric
- C4, C6: value 22uF -> 100nF; footprint Capacitor_SMD:C_0805_2012Metric -> Capacitor_SMD:C_0603_1608Metric
- J1, JP3, JP5: moved to B.Cu
- J2: value USB_C_Receptacle_USB2.0_16P -> Conn_01x06; footprint Connector_USB:USB_C_Receptacle_GCT_USB4105-xx-A_16P_TopMnt_Horizontal -> Connector_JST:JST_GH_SM06B-GHS-TB_1x06-1MP_P1.25mm_Horizontal
- J3: value Conn_02x09_Odd_Even -> Conn_01x02; footprint Connector_PinHeader_2.54mm:PinHeader_2x09_P2.54mm_Horizontal -> Connector_PinHeader_2.00mm:PinHeader_1x02_P2.00mm_Vertical; moved to B.Cu
- R16: value 5.1K -> 47R; moved to F.Cu
- R17: value 5.1K -> 10K; moved to F.Cu
- moved R8 66.7 mm to (128.1, 125.4), turned to -90 degrees
- moved R11 65.0 mm to (129.9, 125.4), turned to -90 degrees
- moved D2 63.7 mm to (128.1, 128.4), turned to 90 degrees
- moved R12 63.3 mm to (131.7, 125.4), turned to -90 degrees
- moved J1 62.0 mm to (130.7, 122.2), turned to -90 degrees
- moved D4 61.9 mm to (129.9, 128.4), turned to 90 degrees
- moved D5 60.1 mm to (131.7, 128.4), turned to 90 degrees
- moved J3 39.7 mm to (121.8, 121.6)
- moved TP3 38.4 mm to (155.0, 116.0)
- moved TP5 37.3 mm to (151.1, 123.4), turned to -135 degrees
- moved TP4 32.6 mm to (149.0, 116.0)
- moved TP2 31.0 mm to (145.0, 120.8)
- moved C25 30.8 mm to (163.0, 94.0)
- moved C6 29.3 mm to (126.8, 120.8), turned to 0 degrees
- moved C17 27.8 mm to (139.1, 121.6), turned to 90 degrees
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Connections:
- net GATE_CLK renamed SPI1_CLK
- net GATE_MISO renamed SPI1_MISO
- net GATE_MOSI renamed SPI1_MOSI
- C34 pad 1: VDC -> GND
- C34 pad 2: GND -> VDC
- C4 pad 1: GND -> NTC_1
- C4 pad 2: VDC -> GND
- C6 pad 1: GND -> NTC_2
- C6 pad 2: VDC -> GND
- H1 pad 1: Net-(H1-Pad1) -> unconnected-(H1-Pad1)
- H2 pad 1: Net-(H1-Pad1) -> unconnected-(H2-Pad1)
- H3 pad 1: Net-(H3-Pad1) -> unconnected-(H3-Pad1)
- H4 pad 1: Net-(H3-Pad1) -> unconnected-(H4-Pad1)
- J3 pad 1: unconnected-(J3-Pin_1-Pad1) -> GND
- J3 pad 2: unconnected-(J3-Pin_2-Pad2) -> NTC_2
- J4 pad S1: unconnected-(J4-PadS1) -> CAN_H
- J4 pad S2: unconnected-(J4-PadS2) -> CAN_L
- J8 pad S1: unconnected-(J8-PadS1) -> CAN_H
- J8 pad S2: unconnected-(J8-PadS2) -> CAN_L
- JP2 pad 1: CAN_H -> CAN_L
- R16 pad 1: GND -> ENCODER2
- R16 pad 2: Net-(J2-CC2) -> Net-(J6-Pin_4)
- R17 pad 1: GND -> NTC_2
- R17 pad 2: Net-(J2-CC1) -> +3.3V
- R19 pad 2: CAN_L -> CAN_H
- U2 pad 22: unconnected-(U2-PC4-Pad22) -> NTC_1
- U2 pad 34: unconnected-(U2-PB12-Pad34) -> LED1
- U2 pad 35: unconnected-(U2-PB13-Pad35) -> LED2
- U2 pad 36: unconnected-(U2-PB14-Pad36) -> LED3
- U2 pad 37: unconnected-(U2-PB15-Pad37) -> NTC_2
- U2 pad 40: unconnected-(U2-PC8-Pad40) -> I2C_SCL
- U2 pad 41: unconnected-(U2-PC9-Pad41) -> I2C_SDA
- U2 pad 43: unconnected-(U2-PA9-Pad43) -> USART1_TX
- U2 pad 44: unconnected-(U2-PA10-Pad44) -> USART1_RX
- U2 pad 55: unconnected-(U2-PD2-Pad55) -> SPI3_CSS
Routing:
- net I2C_SCL: track 0.00 -> 38.2 mm, vias 0 -> 2
- net I2C_SDA: track 0.00 -> 36.6 mm, vias 0 -> 2
- net USART1_TX: track 0.00 -> 33.2 mm, vias 0 -> 2
- net USART1_RX: track 0.00 -> 31.2 mm, vias 0 -> 2
- net CAN_H: track 0.00 -> 28.3 mm
- net ENCODER2: track 0.00 -> 27.0 mm, vias 0 -> 2
- net CAN_L: track 0.00 -> 25.1 mm
- net NTC_2: track 0.00 -> 24.7 mm, vias 0 -> 1
- net ENCODER1: track 0.00 -> 22.3 mm, vias 0 -> 2
- net LED3: track 0.00 -> 22.0 mm, vias 0 -> 2
- net LED2: track 0.00 -> 21.9 mm, vias 0 -> 2
- net LED1: track 0.00 -> 21.8 mm, vias 0 -> 2
- net +3.3V: track 27.3 -> 47.4 mm, vias 10 -> 17
- net NTC_1: track 0.00 -> 20.1 mm, vias 0 -> 1
- net VBUS: track 0.00 -> 17.8 mm, vias 0 -> 1
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- added copper zone on F.Cu, net +5V
- added copper zone on In2.Cu, net +5V
- added copper zone on B.Cu, net unconnected-(H1-Pad1)
- added copper zone on F.Cu, net unconnected-(H1-Pad1)
- added copper zone on B.Cu, net unconnected-(H2-Pad1)
- added copper zone on F.Cu, net unconnected-(H2-Pad1)
- added copper zone on B.Cu, net unconnected-(H3-Pad1)
- added copper zone on F.Cu, net unconnected-(H3-Pad1)
- added copper zone on B.Cu, net unconnected-(H4-Pad1)
- added copper zone on F.Cu, net unconnected-(H4-Pad1)
- removed copper zone on In2.Cu, net GND
Other:
- board text added: "CANR"
- board text added: "CLK"
- board text added: "GND"
- board text added: "NTC"

Commit message: update
Parts:
- added TP9: TestPoint, TestPoint:TestPoint_Pad_D1.0mm, B.Cu at (147.8, 108.8)
- C10: moved to B.Cu
- moved TP7 9.42 mm to (151.1, 104.3)
- moved TP6 6.71 mm to (151.1, 106.3)
- moved C10 5.64 mm to (142.6, 108.5), turned to 0 degrees
- moved TP8 4.18 mm to (151.1, 108.3)
- moved TP3 3.00 mm to (152.0, 116.0), turned to 90 degrees
- moved R9 2.11 mm to (138.6, 117.8)
- moved R10 1.24 mm to (155.9, 100.9)
- moved C4 1.24 mm to (152.9, 100.9)
- moved C21 0.61 mm to (146.1, 105.2)
Connections:
- R13 pad 1: BOOT -> CANRX
- U1 pad 8: unconnected-(U1-CS-Pad8) -> ENCODER_CS
- U2 pad 17: unconnected-(U2-PA3-Pad17) -> ENCODER_CS
- U2 pad 45: D- -> CANRX
- U2 pad 46: D+ -> CANTX
- U2 pad 62: CANTX -> unconnected-(U2-PB9-Pad62)
- U2 pad 8: unconnected-(U2-PC0-Pad8) -> GATE_CS
Routing:
- net GATE_CS: track 2.17 -> 15.0 mm, vias 0 -> 2
- net ENCODER_CS: track 0.00 -> 10.3 mm, vias 0 -> 1
- net CANRX: track 0.00 -> 7.81 mm, vias 0 -> 2
- net SPI1_MISO: track 33.4 -> 25.8 mm
- net SPI1_MOSI: track 31.4 -> 25.1 mm
- net SPI1_CLK: track 26.4 -> 21.5 mm
- net VDC: track 13.5 -> 10.8 mm, vias 133 -> 134
- net NTC_1: track 20.1 -> 22.7 mm
- net BOOT: track 8.48 -> 5.97 mm
- net SWDIO: track 10.2 -> 8.31 mm
- net +3.3V: track 47.4 -> 45.8 mm
- net Net-(Q4-G): track 34.5 -> 33.9 mm
- net SPC: track 30.3 -> 29.8 mm
- net CANTX: track 9.65 -> 10.2 mm, vias 0 -> 2
- net GND: track 0.98 -> 0.92 mm, vias 134 -> 156
- added copper zone on F.Cu, net +3.3V
- added copper zone on In2.Cu, net GND
Other:
- board text added: "+"
- board text added: "3V3"
- board text added: "5V"
- board text added: "BOOT"
- board text added: "CSS"
- board text added: "DIO"
- board text added: "H"
- board text added: "L"
- board text added: "MISO"
- board text added: "MOSI"
- board text added: "RST"
- board text added: "U"
- board text added: "V"
- board text added: "W"
