File: PCB/foc-motor-controller.kicad_pcb (KiCad board)
At the start: 4 copper layers, 50 x 50 mm, 118 parts, among them J1 SWD, J2 Conn_01x06, J3 Conn_01x02, J4 XT30PW_2_2_-M.G.B, J6 Conn_01x08, J8 XT30PW_2_2_-M.G.B, Q1 DON50N04, Q2 DON50N04, Q3 DON50N04, Q4 NMOS-8PINS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

Commit message: clean up schematic
Parts:
- removed D2, D4, D5: LED_Small, LED_SMD:LED_0603_1608Metric
- removed JP3: SolderJumper_2_Open, Jumper:SolderJumper-2_P1.3mm_Open_RoundedPad1.0x1.5mm
- removed JP5: SolderJumper_2_Open, Jumper:SolderJumper-2_P1.3mm_Open_TrianglePad1.0x1.5mm
- added C35: 2.2nF, Capacitor_SMD:C_0603_1608Metric, B.Cu at (146.5, 109.3)
- added C46: 2.2nF, Capacitor_SMD:C_0603_1608Metric, F.Cu at (147.6, 105.5)
- added C47: 2.2nF, Capacitor_SMD:C_0603_1608Metric, B.Cu at (145.0, 109.2)
- added C48: 10uF, Capacitor_SMD:C_1206_3216Metric, F.Cu at (132.7, 94.0)
- added C49: 10uF, Capacitor_SMD:C_1206_3216Metric, F.Cu at (135.0, 94.0)
- added C50: 10uF, Capacitor_SMD:C_1206_3216Metric, F.Cu at (137.3, 94.0)
- added C51: 10uF, Capacitor_SMD:C_1206_3216Metric, F.Cu at (146.7, 94.0)
- added C52: 10uF, Capacitor_SMD:C_1206_3216Metric, F.Cu at (149.0, 94.0)
- added C53: 10uF, Capacitor_SMD:C_1206_3216Metric, F.Cu at (151.3, 94.0)
- added C54: 10uF, Capacitor_SMD:C_1206_3216Metric, F.Cu at (160.7, 94.0)
- added C55: 10uF, Capacitor_SMD:C_1206_3216Metric, F.Cu at (163.0, 94.0)
- added C56: 10uF, Capacitor_SMD:C_1206_3216Metric, F.Cu at (165.3, 94.0)
- added D6: LED_RBAG, LED_SMD:LED_Cree-PLCC4_2x2mm_CW, F.Cu at (129.9, 128.5)
- added RN2: 56R, Resistor_SMD:R_Array_Convex_4x0402, F.Cu at (151.8, 107.5)
- C18, C30: value 10uF -> 22uF
- C22, C25, C40: value C_Polarized -> 47uF
- J2: value Conn_01x06 -> SPI
- J6: value Conn_01x08 -> COMMS
- L2: value 12uH -> 47uH
- R3: value 1K -> 237K
- R4: value 115K -> 52.3K
- moved C10 1.20 mm to (143.5, 109.3), turned to -90 degrees
- moved TP9 0.90 mm to (148.7, 108.8)
- moved G*** 0.70 mm to (152.7, 117.7)
- moved C36 0.22 mm to (152.3, 109.5)
- moved R18 0.10 mm to (152.2, 112.4)
- moved R20 0.10 mm to (153.7, 112.4)
- moved R21 0.10 mm to (155.2, 112.4)
Connections:
- net GATE_CS renamed DRIVER_CS
- R18 pad 1: GATE_FAULT -> DRIVER_FAULT
- R25 pad 2: GATE_EN -> DRIVER_EN
- U1 pad 4: unconnected-(U1-CAL_EN-Pad4) -> ENC_CAL
- U2 pad 26: unconnected-(U2-PB2-Pad26) -> ENC_CAL
- U2 pad 3: unconnected-(U2-PC14-Pad3) -> DRIVER_FAULT
- U2 pad 4: unconnected-(U2-PC15-Pad4) -> DRIVER_EN
- U3 pad 21: CURR_SENSE_C -> Net-(RN2B-R2.2)
- U3 pad 22: CURR_SENSE_B -> Net-(RN2C-R3.2)
- U3 pad 23: CURR_SENSE_A -> Net-(RN2D-R4.2)
- U3 pad 25: GATE_FAULT -> DRIVER_FAULT
- U3 pad 30: GATE_EN -> DRIVER_EN
Routing:
- net DRIVER_EN: track 0.00 -> 23.2 mm, vias 0 -> 2
- net DRIVER_FAULT: track 0.00 -> 20.1 mm, vias 0 -> 2
- net ENC_CAL: track 0.00 -> 17.0 mm, vias 0 -> 1
- net unconnected-(U1-CAL_EN-Pad4): track 15.8 -> 0.00 mm
- net GATE_FAULT: track 4.59 -> 0.00 mm
- net CURR_SENSE_C: track 10.6 -> 7.83 mm
- net CURR_SENSE_A: track 11.3 -> 8.56 mm, vias 0 -> 1
- net +3.3V: track 44.8 -> 47.5 mm, vias 17 -> 18
- net Net-(RN2D-R4.2): track 0.00 -> 2.42 mm
- net SPI1_CLK: track 21.5 -> 19.3 mm
- net Net-(RN2C-R3.2): track 0.00 -> 2.01 mm
- net Net-(D6-GK): track 1.39 -> 3.19 mm
- net Net-(RN2B-R2.2): track 0.00 -> 1.60 mm
- net SPI1_MISO: track 25.8 -> 24.3 mm
- net CURR_SENSE_B: track 11.0 -> 9.48 mm, vias 0 -> 1
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
Commit message: update
Parts:
- moved G*** 0.40 mm to (152.7, 118.1)
Connections:
- net GATE_CAL renamed DRIVER_CAL
Routing:
- net +3.3V: track 47.5 -> 46.2 mm
- net NTC_2: track 24.6 -> 25.5 mm
- net VBUS: track 17.8 -> 18.4 mm
- net DRIVER_FAULT: track 20.1 -> 19.5 mm
- net SPI1_MISO: track 24.3 -> 23.7 mm
- net DRIVER_EN: track 23.2 -> 22.7 mm
- net MOTOR_OUT_2: track 18.7 -> 18.3 mm, vias 90 -> 43
- net MOTOR_OUT_3: track 31.6 -> 31.4 mm, vias 90 -> 43
- net MOTOR_OUT_1: track 13.8 -> 13.7 mm, vias 90 -> 43
- net GND: vias 176 -> 179
- added copper zone on In1.Cu, net unconnected-(H1-Pad1)
- added copper zone on In2.Cu, net unconnected-(H1-Pad1)
- added copper zone on In1.Cu, net unconnected-(H2-Pad1)
- added copper zone on In2.Cu, net unconnected-(H2-Pad1)
- added copper zone on In1.Cu, net unconnected-(H3-Pad1)
- added copper zone on In2.Cu, net unconnected-(H3-Pad1)
- added copper zone on In1.Cu, net unconnected-(H4-Pad1)
- added copper zone on In2.Cu, net unconnected-(H4-Pad1)
