File: PCB/foc-motor-controller-rounded.kicad_pcb (KiCad board)
At the start: 4 copper layers, 50 x 50 mm, 118 parts, among them J1 SWD, J2 Conn_01x06, J3 Conn_01x02, J4 XT30PW_2_2_-M.G.B, J6 Conn_01x08, J8 XT30PW_2_2_-M.G.B, Q1 DON50N04, Q2 DON50N04, Q3 DON50N04, Q4 NMOS-8PINS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

Commit message: update
Parts:
- added C35: 2.2nF, Capacitor_SMD:C_0603_1608Metric, B.Cu at (145.0, 109.3)
- added C46: 2.2nF, Capacitor_SMD:C_0603_1608Metric, F.Cu at (147.5, 105.7)
- added C47: 2.2nF, Capacitor_SMD:C_0603_1608Metric, B.Cu at (146.5, 109.3)
- added C48: 10uF, Capacitor_SMD:C_1206_3216Metric, F.Cu at (146.7, 94.0)
- added C49: 10uF, Capacitor_SMD:C_1206_3216Metric, F.Cu at (149.0, 94.0)
- added C50: 10uF, Capacitor_SMD:C_1206_3216Metric, F.Cu at (151.3, 94.0)
- added C51: 10uF, Capacitor_SMD:C_1206_3216Metric, F.Cu at (160.7, 94.0)
- added C52: 10uF, Capacitor_SMD:C_1206_3216Metric, F.Cu at (163.0, 94.0)
- added C53: 10uF, Capacitor_SMD:C_1206_3216Metric, F.Cu at (165.3, 94.0)
- added C54: 10uF, Capacitor_SMD:C_1206_3216Metric, F.Cu at (132.7, 94.0)
- added C55: 10uF, Capacitor_SMD:C_1206_3216Metric, F.Cu at (135.0, 94.0)
- added C56: 10uF, Capacitor_SMD:C_1206_3216Metric, F.Cu at (137.3, 94.0)
- added RN2: 56R, Resistor_SMD:R_Array_Convex_4x0402, F.Cu at (151.7, 107.6)
- C18, C30: value 10uF -> 22uF
- C22, C25, C40: value C_Polarized -> 47uF
- L2: value 12uH -> 47uH
- R3: value 1K -> 237K
- R4: value 115K -> 52.3K
- moved C10 1.20 mm to (143.5, 109.3), turned to -90 degrees
- moved TP9 1.10 mm to (148.9, 108.9)
- moved C36 0.36 mm to (152.2, 109.6)
- moved C21 0.20 mm to (145.9, 105.2)
Connections:
- U1 pad 4: unconnected-(U1-CAL_EN-Pad4) -> ENC_CAL
- U2 pad 26: unconnected-(U2-PB2-Pad26) -> ENC_CAL
- U3 pad 21: CURR_SENSE_C -> Net-(RN2B-R2.2)
- U3 pad 22: CURR_SENSE_B -> Net-(RN2C-R3.2)
- U3 pad 23: CURR_SENSE_A -> Net-(RN2D-R4.2)
Routing:
- net ENC_CAL: track 0.00 -> 18.3 mm, vias 0 -> 1
- net unconnected-(U1-CAL_EN-Pad4): track 15.8 -> 0.00 mm
- net CURR_SENSE_C: track 10.6 -> 7.77 mm
- net CURR_SENSE_A: track 11.3 -> 8.55 mm, vias 0 -> 1
- net Net-(RN2D-R4.2): track 0.00 -> 2.57 mm
- net Net-(RN2C-R3.2): track 0.00 -> 2.15 mm
- net CURR_SENSE_B: track 11.0 -> 9.05 mm, vias 0 -> 1
- net Net-(RN2B-R2.2): track 0.00 -> 1.74 mm
- net SPI1_CLK: track 21.5 -> 20.0 mm
- net +3.3V: track 44.8 -> 46.0 mm
- net GND: vias 182 -> 177
Other:
- board text added: "CS"
- board text removed: "CSS"
