File: PCB/foc-motor-controller.kicad_sch (KiCad schematic)
At the start: 103 parts, among them J1 SWD, J2 USB_C_Receptacle_USB2.0_16P, J3 Conn_02x09_Odd_Even, J4 XT30PW_2_2_-M.G.B, J6 CAN_OUT, J7 CAN_IN, J8 XT30PW_2_2_-M.G.B, J9 Conn_01x05, Q1 DON50N04, Q2 DON50N04, Q3 DON50N04, Q4 NMOS-8PINS, Q5 DON50N04, Q6 DON50N04, U1 MT6826SGT, U2 STM32G431RBTx, U3 DRV8323SRTAT, U4 MIC5219-3.3YM5, U5 TCAN1044V, U6 USBLC6-2SC6, U7 TPS54240DGQ, Y1 Resonator

Commit message: update
Parts:
- removed C22, C25, C34: 470uF, Capacitor_SMD:C_Elec_10x10.2, symbol Device:C_Polarized_Small
- removed C35, C4, C6: 22uF, Capacitor_SMD:C_0805_2012Metric, symbol Device:C
- removed J2: USB_C_Receptacle_USB2.0_16P, Connector_USB:USB_C_Receptacle_GCT_USB4105-xx-A_16P_TopMnt_Horizontal, symbol Connector:USB_C_Receptacle_USB2.0_16P
- removed J3: Conn_02x09_Odd_Even, Connector_PinHeader_2.54mm:PinHeader_2x09_P2.54mm_Horizontal, symbol Connector_Generic:Conn_02x09_Odd_Even
- removed J6: CAN_OUT, Connector_JST:JST_GH_SM04B-GHS-TB_1x04-1MP_P1.25mm_Horizontal, symbol Connector_Generic:Conn_01x04
- removed J7: CAN_IN, Connector_JST:JST_GH_SM04B-GHS-TB_1x04-1MP_P1.25mm_Horizontal, symbol Connector_Generic:Conn_01x04
- removed J9: Conn_01x05, TiManh:TerminalBlock_1x05_P6.35mm_Horizontal, symbol Connector_Generic:Conn_01x05
- removed U6: USBLC6-2SC6, Package_TO_SOT_SMD:SOT-23-6, symbol Power_Protection:USBLC6-2SC6
- added C12, C20, C4, C6: 100nF, Capacitor_SMD:C_0603_1608Metric, symbol Device:C_Small
- added C22, C25, C40: C_Polarized, Capacitor_SMD:CP_Elec_6.3x5.9, symbol Device:C_Polarized
- added C34, C41, C42, C43, C44, C45: 10uF, Capacitor_SMD:C_1206_3216Metric, symbol Device:C
- added D3: D_TVS, Diode_SMD:D_SMB, symbol Device:D_TVS
- added J2: Conn_01x06, Connector_JST:JST_GH_SM06B-GHS-TB_1x06-1MP_P1.25mm_Horizontal, symbol Connector_Generic:Conn_01x06
- added J3: Conn_01x02, Connector_PinHeader_2.00mm:PinHeader_1x02_P2.00mm_Vertical, symbol Connector_Generic:Conn_01x02
- added J6: Conn_01x08, Connector_JST:JST_GH_SM08B-GHS-TB_1x08-1MP_P1.25mm_Horizontal, symbol Connector_Generic:Conn_01x08
- added R10: 10K, Resistor_SMD:R_0603_1608Metric, symbol Device:R_Small
- added R27: 47R, Resistor_SMD:R_0603_1608Metric, symbol Device:R_Small
- added R28, R29: 4.7K, Resistor_SMD:R_0603_1608Metric, symbol Device:R_Small
- added TH1: Thermistor_NTC, Resistor_SMD:R_0603_1608Metric, symbol Device:Thermistor_NTC
- added TP6, TP7, TP8: TestPoint, TestPoint:TestPoint_Pad_D1.0mm, symbol Connector:TestPoint
- R16: value 5.1K -> 47R
- R17: value 5.1K -> 10K
Connections:
- net +3.3V: now also R17.2, R10.2, R28.2, R29.2
- net CAN_H: now also J4.S1, J8.S1, R19.2; no longer JP2.1 (A)
- net CAN_L: now also J4.S2, J8.S2, JP2.1 (A); no longer R19.2
- net ENCODER1: now also C12.1, R27.1
- net ENCODER2: now also R16.1, C20.1
- net GND: now also C12.2, C20.2, C22.2, C25.2, C34.1, C4.2, C40.2, C41.1, C42.1, C43.1, C44.1, C45.1, C6.2, D3.2 (A2), J2.1 (Pin_1), J3.1 (Pin_1), J6.1 (Pin_1), TH1.2; no longer R16.1, R17.1
- net LED1: now also U2.34 (PB12)
- net LED2: now also U2.35 (PB13)
- net LED3: now also U2.36 (PB14)
- net SPI3_CLK: now also J2.4 (Pin_4)
- net SPI3_MISO: now also J2.6 (Pin_6)
- net SPI3_MOSI: now also J2.5 (Pin_5)
- net VBUS: now also J2.2 (Pin_2), J6.2 (Pin_2)
- net VDC: now also C22.1, C25.1, C34.2, C40.1, C41.2, C42.2, C43.2, C44.2, C45.2, D3.1 (A1)
- net at H4.1: no longer H3.1
- net NTC_1: now reaches U2.22 (PC4)
- net NTC_1: now also C4.1, R10.1, TH1.1
- net NTC_2: now reaches U2.37 (PB15)
- net NTC_2: now also R17.1, C6.1, J3.2 (Pin_2)
- net I2C_SCL: now reaches U2.40 (PC8)
- net I2C_SCL: now also J6.8 (Pin_8), R28.1
- net I2C_SDA: now reaches U2.41 (PC9)
- net I2C_SDA: now also J6.7 (Pin_7), R29.1
- net USART1_TX: now reaches U2.43 (PA9)
- net USART1_TX: now also J6.6 (Pin_6)
- net USART1_RX: now reaches U2.44 (PA10)
- net USART1_RX: now also J6.5 (Pin_5)
- net SPI3_CSS: now reaches U2.55 (PD2)
- net SPI3_CSS: now also J2.3 (Pin_3)
- net at R16.2: now also J6.4 (Pin_4)
- net at H2.1: no longer H1.1
- net GATE_CLK renamed SPI1_CLK
- net SPI1_CLK: now also TP8.1
- net GATE_MISO renamed SPI1_MISO
- net SPI1_MISO: now also TP7.1
- net GATE_MOSI renamed SPI1_MOSI
- net SPI1_MOSI: now also TP6.1
- new net: J6.3 (Pin_3), R27.2
- no-connect marks 1 -> 0
Other:
- moved on the sheet: H1, H2, H3, H4, J4, J8, JP2, JP5, R19, R21, TP4, TP5

Commit message: update
Parts:
- added TP9: TestPoint, TestPoint:TestPoint_Pad_D1.0mm, symbol Connector:TestPoint
Connections:
- net D+ is gone; now on net CANTX: U2.46 (PA12)
- net BOOT: no longer R13.1
- net CANTX: no longer U2.62 (PB9)
- net GATE_CS: now also U2.8 (PC0)
- net ENCODER_CS: now reaches U2.17 (PA3)
- net ENCODER_CS: now also U1.8 (CS), TP9.1
- net D- renamed CANRX
- net CANRX: now also R13.1
Other:
- moved on the sheet: C34, C37, C38, C39, C41, C42, C43, C44, C45, Q1, Q2, Q3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

Commit message: update
Parts:
- added C35, C46, C47: 2.2nF, Capacitor_SMD:C_0603_1608Metric, symbol Device:C_Small
- added C48, C49, C50, C51, C52, C53, C54, C55, C56: 10uF, Capacitor_SMD:C_1206_3216Metric, symbol Device:C
- added RN2: 56R, Resistor_SMD:R_Array_Convex_4x0402, symbol Device:R_Pack04_Split
- C18, C30: value 10uF -> 22uF
- C22, C25, C40: value C_Polarized -> 47uF; now not fitted
- L2: value 12uH -> 47uH
- R3: value 1K -> 237K
- R4: value 115K -> 52.3K
Connections:
- net CURR_SENSE_A: now also C47.2, RN2.4 (R4.1); no longer U3.23 (SOA)
- net CURR_SENSE_B: now also C35.2, RN2.3 (R3.1); no longer U3.22 (SOB)
- net CURR_SENSE_C: now also C46.2, RN2.2 (R2.1); no longer U3.21 (SOC)
- net GATE_CAL: now also U2.2 (PC13)
- net GND: now also C35.1, C46.1, C47.1, C48.1, C49.1, C50.1, C51.1, C52.1, C53.1, C54.1, C55.1, C56.1
- net VDC: now also C48.2, C49.2, C50.2, C51.2, C52.2, C53.2, C54.2, C55.2, C56.2
- net ENC_CAL: now reaches U2.26 (PB2)
- net ENC_CAL: now also U1.4 (CAL_EN)
- new net: RN2.5 (R4.2), U3.23 (SOA)
- new net: RN2.6 (R3.2), U3.22 (SOB)
- new net: RN2.7 (R2.2), U3.21 (SOC)
Other:
- note added: "Optional capacitors (polymer vs ceramic)"
- moved on the sheet: C10, C12, C20, C34, C36, C41, C42, C43, C44, C45, D3, J6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

Commit message: clean up schematic
Parts:
- removed D2, D4, D5: LED_Small, LED_SMD:LED_0603_1608Metric, symbol Device:LED_Small
- removed JP3: SolderJumper_2_Open, Jumper:SolderJumper-2_P1.3mm_Open_RoundedPad1.0x1.5mm, symbol Jumper:SolderJumper_2_Open
- removed JP5: SolderJumper_2_Open, Jumper:SolderJumper-2_P1.3mm_Open_TrianglePad1.0x1.5mm, symbol Jumper:SolderJumper_2_Open
- added D6: LED_RBAG, LED_SMD:LED_Cree-PLCC4_2x2mm_CW, symbol Device:LED_RBAG
- J2: value Conn_01x06 -> SPI
- J6: value Conn_01x08 -> COMMS
- JP2, TP3, TP4, TP5, TP8: now left out of the parts list
Connections:
- net GATE_EN is gone; now on net DRIVER_EN: R25.2, U3.30 (ENABLE)
- net GATE_FAULT is gone; now on net DRIVER_FAULT: R18.1, U3.25 (FAULT_N)
- net +3.3V: now also D6.3 (A)
- net at R11.2: now also D6.4 (GK)
- net at R8.2: now also D6.1 (RK)
- net at R12.2: now also D6.2 (BK)
- net DRIVER_FAULT: now reaches U2.3 (PC14)
- net DRIVER_EN: now reaches U2.4 (PC15)
- net GATE_CAL renamed DRIVER_CAL
- net GATE_CS renamed DRIVER_CS
- no-connect marks 0 -> 25
Other:
- note added: "Bulk capacitors (polymer or ceramic)"
- note added: "CONN"
- note added: "DRIVER"
- note added: "ENCODER"
- note added: "NTC"
- note removed: "Optional capacitors (polymer vs ceramic)"
- moved on the sheet: C1, C10, C11, C12, C13, C14, C15, C16, C17, C18, C19, C2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

Commit message: update
Connections:
- no-connect marks 25 -> 21
Other:
- moved on the sheet: C28, C29, C31, JP2, R13, R14, R19, U5
