File: PCB/G4-FOC-Driver.kicad_pcb (KiCad board)
At the start: 4 copper layers, 50 x 50 mm, 127 parts, among them J1 SWD, J2 SPI, J3 Conn_01x02, J4 XT30PW_2_2_-M.G.B, J6 COMMS, J8 XT30PW_2_2_-M.G.B, Q1 DON50N04, Q2 DON50N04, Q3 DON50N04, Q4 NMOS-8PINS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

Commit message: update
Parts:
- C11, C14: value 100nF -> 47nF
- Q1, Q2, Q3, Q5, Q6: value DON50N04 -> NMOS-8PINS
- R15: value 1K -> 10K
