File: PCB/G4-FOC-Driver.kicad_sch (KiCad schematic)
At the start: 126 parts, among them J1 SWD, J2 SPI, J3 Conn_01x02, J4 XT30PW_2_2_-M.G.B, J6 COMMS, J8 XT30PW_2_2_-M.G.B, Q1 DON50N04, Q2 DON50N04, Q3 DON50N04, Q4 NMOS-8PINS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

Commit message: clean up schematic
Parts:
- Q1, Q2, Q3, Q5, Q6: value DON50N04 -> NMOS-8PINS
Changed lines of the file:
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@@
 			)
 		)
-		(property "Value" "DON50N04"
+		(property "Value" "NMOS-8PINS"
 			(at 382.778 54.864 0)
 			(effects
@@
 			)
 		)
-		(property "Value" "DON50N04"
+		(property "Value" "NMOS-8PINS"
 			(at 385.318 82.55 0)
 			(effects
@@
 			)
 		)
-		(property "Value" "DON50N04"
+		(property "Value" "NMOS-8PINS"
 			(at 365.252 74.422 0)
 			(effects
@@
 			)
 		)
-		(property "Value" "DON50N04"
+		(property "Value" "NMOS-8PINS"
 			(at 383.54 43.434 0)
 			(effects
@@
 			)
 		)
-		(property "Value" "DON50N04"
+		(property "Value" "NMOS-8PINS"
 			(at 366.014 63.754 0)
 			(effects

Commit message: update
Parts:
- C11, C14: value 100nF -> 47nF
- R15: value 1K -> 10K
Changed lines of the file:
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@@
 			)
 		)
-		(property "Value" "100nF"
+		(property "Value" "47nF"
 			(at 74.93 93.9799 0)
 			(effects
@@
 			)
 		)
-		(property "Value" "100nF"
+		(property "Value" "47nF"
 			(at 87.63 97.7899 0)
 			(effects
@@
 			)
 		)
-		(property "Value" "1K"
+		(property "Value" "10K"
 			(at 86.36 90.17 90)
 			(effects
